File: schematics/cpu.sch (KiCad schematic (older format))
At the start: 75 parts

Commit message: updated schema
Parts:
- added Diesel_safety_relay: ??, Relay_THT:Relay_StandexMeder_DIP_LowProfile, symbol Relay:DIPxx-1Axx-11x
- added Diesel_valve: 80mA, symbol Device:L
- added Diesel_valve_relay, Electric_heater: К293КП11Б, Relay_THT:Relay_StandexMeder_DIP_LowProfile, symbol Relay:DIPxx-1Axx-11x
- added R? (x2): 360, symbol Device:R
- added R?: 500k, symbol Device:R
- added U?: ULN2003, symbol Transistor_Array:ULN2003
- EHeat+pump: renamed from Furnace_pump; value UPS 60W 270mA -> relays + UPS 60W 300mA
- renumbered Furnace to Furnace+relay, Furnace_valve to Pump_valve
Connections:
- wire segments 359 -> 411
Other:
- note added: "Heater circuit, separate power line"

Commit message: K293KP11B proved unreliable on currents over 1A with radiator pump. after replacing two optrons decided to fallback to regular relay for radiator pump circuit. note 360Ohm in control line removed or shortened in this case
Parts:
- removed R?: 360, symbol Device:R
- removed Radiator_relay: К293КП11Б, Relay_THT:Relay_StandexMeder_DIP_LowProfile, symbol Relay:DIPxx-1Axx-11x
- added Radiator_pump_relay: RE030005, Relay_THT:Relay_StandexMeder_DIP_LowProfile, symbol Relay:DIPxx-1Axx-11x
Connections:
- wire segments 411 -> 410
Changed lines of the file:
@@
 	9400 3400 10300 3400
-$Comp
-L Relay:DIPxx-1Axx-11x Radiator_relay
-U 1 1 5B832597
-P 7850 3100
-F 0 "Radiator_relay" H 8180 3146 50  0000 L CNN
-F 1 "К293КП11Б" H 8180 3055 50  0000 L CNN
-F 2 "Relay_THT:Relay_StandexMeder_DIP_LowProfile" H 8200 3050 50  0001 L CNN
-F 3 "https://standexelectronics.com/wp-content/uploads/datasheet_reed_relay_DIP.pdf" H 7850 3100 50  0001 C CNN
-	1    7850 3100
-	1    0    0    -1
-$EndComp
 $Comp
 L Relay:DIPxx-1Axx-11x Furnace_relay
@@
 F 3 "~" H 5550 7350 50  0001 C CNN
 	1    5550 7350
-	-1   0    0    1
-$EndComp
-$Comp
-L Device:R R?
-U 1 1 5B9D0D76
-P 5650 7700
-F 0 "R?" V 5443 7700 50  0000 C CNN
-F 1 "360" V 5534 7700 50  0000 C CNN
-F 2 "" V 5580 7700 50  0001 C CNN
-F 3 "~" H 5650 7700 50  0001 C CNN
-	1    5650 7700
 	-1   0    0    1
 $EndComp
@@
 	5550 7200 5550 5050
 Wire Wire Line
-	5650 7550 5650 5150
-Wire Wire Line
 	4750 7800 4750 8800
 Wire Wire Line
@@
 	5550 7500 5550 9900
 Wire Wire Line
-	5650 7850 5650 10000
-Wire Wire Line
 	1100 3500 1100 9500
 Wire Wire Line
@@
 Wire Wire Line
 	9400 1400 9400 1450
+$Comp
+L Relay:DIPxx-1Axx-11x Radiator_pump_relay
+U 1 1 68CF24BE
+P 7850 3100
+F 0 "Radiator_pump_relay" H 8180 3146 50  0000 L CNN
+F 1 "RE030005 " H 8180 3055 50  0000 L CNN
+F 2 "Relay_THT:Relay_StandexMeder_DIP_LowProfile" H 8200 3050 50  0001 L CNN
+F 3 "https://standexelectronics.com/wp-content/uploads/datasheet_reed_relay_DIP.pdf" H 7850 3100 50  0001 C CNN
+	1    7850 3100
+	1    0    0    -1
+$EndComp
+Wire Wire Line
+	5650 5150 5650 10000
 $EndSCHEMATC
